File: Hub/DB9toUSB1.sch (KiCad schematic (older format))
At the start: 21 parts, among them J1 Conn_02x03_Odd_Even, J2 Joy1, J3 Joy1, J6 Joy1, SW1 328RST, U1 ATmega328P-AU, X1 12MHz

Commit message: add some missing data / add forgotten pullup for ESP32
Connections:
- wire segments 117 -> 113
Changed lines of the file:
@@
 $Descr A4 11693 8268
 encoding utf-8
-Sheet 2 8
+Sheet 2 7
 Title "MiSTer USB HUB DB9"
 Date "2018-07-31"
@@
 NoConn ~ 4700 3500
 NoConn ~ 4700 3400
-Wire Wire Line
-	4700 3000 5100 3000
 Wire Wire Line
 	6450 3000 6450 3400
@@
 AT328_1_PB5
 Wire Wire Line
-	5100 3000 6450 3000
-Wire Wire Line
-	5100 3100 5100 3200
-Wire Wire Line
 	5100 2600 5100 3000
 Wire Wire Line
 	4700 3100 5100 3100
-Wire Wire Line
-	5100 3200 5100 3300
-Wire Wire Line
-	5100 3300 5100 3650
 Wire Wire Line
 	4700 3200 5100 3200
@@
 Wire Wire Line
 	7150 5200 7400 5200
-Connection ~ 5100 3000
-Wire Wire Line
-	5100 3000 5100 3100
-Connection ~ 5100 3100
 Wire Wire Line
 	5100 3100 6250 3100
-Connection ~ 5100 3200
 Wire Wire Line
 	5100 3200 6950 3200
-Connection ~ 5100 3300
 Wire Wire Line
 	5100 3300 5750 3300
+Wire Wire Line
+	4700 3000 6450 3000
+Wire Wire Line
+	5100 3000 5100 3650
 $EndSCHEMATC
