File: Hub/USBHubPower.sch (KiCad schematic (older format))
At the start: 18 parts, among them J13 Barrel_Jack, U3 Terminus_Technology_FE2.1

Commit message: add some missing data / add forgotten pullup for ESP32
Parts:
- gave numbers to parts that had none: 5
Connections:
- net labels added: FE_2_1_RST, VDD3_3_FE21
Changed lines of the file:
@@
 $Descr A4 11693 8268
 encoding utf-8
-Sheet 5 8
+Sheet 5 7
 Title "MiSTer USB HUB DB9"
 Date "2018-07-31"
@@
 L power:GND #PWR038
 U 1 1 5B34EF4A
-P 5800 1800
-F 0 "#PWR038" H 5800 1550 50  0001 C CNN
-F 1 "GND" H 5800 1650 50  0000 C CNN
-F 2 "" H 5800 1800 50  0001 C CNN
-F 3 "" H 5800 1800 50  0001 C CNN
-	1    5800 1800
+P 5750 2100
+F 0 "#PWR038" H 5750 1850 50  0001 C CNN
+F 1 "GND" H 5750 1950 50  0000 C CNN
+F 2 "" H 5750 2100 50  0001 C CNN
+F 3 "" H 5750 2100 50  0001 C CNN
+	1    5750 2100
 	1    0    0    -1
 $EndComp
@@
 P 7750 5750
 AR Path="/5B3365B6/5BBA4B99" Ref="X?"  Part="1"
-AR Path="/5B3365B0/5BBA4B99" Ref="X?"  Part="1"
-F 0 "X?" V 7900 5750 50  0000 C CNN
+AR Path="/5B3365B0/5BBA4B99" Ref="X3"  Part="1"
+F 0 "X3" V 7900 5750 50  0000 C CNN
 F 1 "12MHz" V 7600 5750 50  0000 C CNN
 F 2 "Crystals:Crystal_SMD_5032-2pin_5.0x3.2mm_HandSoldering" H 7750 5750 50  0001 C CNN
@@
 P 4100 5400
 AR Path="/5B3365B6/5BBA4BA5" Ref="#PWR?"  Part="1"
-AR Path="/5B3365B0/5BBA4BA5" Ref="#PWR?"  Part="1"
-F 0 "#PWR?" H 4100 5250 50  0001 C CNN
+AR Path="/5B3365B0/5BBA4BA5" Ref="#PWR0105"  Part="1"
+F 0 "#PWR0105" H 4100 5250 50  0001 C CNN
 F 1 "+3.3V" H 4100 5540 50  0000 C CNN
 F 2 "" H 4100 5400 50  0001 C CNN
@@
 P 5850 5750
 AR Path="/5B3365B6/5BBA4BAC" Ref="U?"  Part="4"
-AR Path="/5B3365B0/5BBA4BAC" Ref="U?"  Part="4"
-F 0 "U?" H 5850 5650 50  0000 C CNN
+AR Path="/5B3365B0/5BBA4BAC" Ref="U3"  Part="4"
+F 0 "U3" H 5850 5650 50  0000 C CNN
 F 1 "Terminus_Technology_FE2.1" H 5850 5850 50  0000 C CNN
 F 2 "Housings_QFP:LQFP-48_7x7mm_Pitch0.5mm" H 5850 5750 50  0001 C CNN
@@
 P 4100 5550
 AR Path="/5B3365B6/5BBA4BB5" Ref="R?"  Part="1"
-AR Path="/5B3365B0/5BBA4BB5" Ref="R?"  Part="1"
-F 0 "R?" H 4159 5596 50  0000 L CNN
+AR Path="/5B3365B0/5BBA4BB5" Ref="R22"  Part="1"
+F 0 "R22" H 4159 5596 50  0000 L CNN
 F 1 "10k" H 4159 5505 50  0000 L CNN
 F 2 "Resistors_SMD:R_0805_HandSoldering" H 4100 5550 50  0001 C CNN
@@
 P 3600 5800
 AR Path="/5B3365B6/5BBA4BBE" Ref="SW?"  Part="1"
-AR Path="/5B3365B0/5BBA4BBE" Ref="SW?"  Part="1"
-F 0 "SW?" H 3600 6067 50  0000 C CNN
+AR Path="/5B3365B0/5BBA4BBE" Ref="SW2"  Part="1"
+F 0 "SW2" H 3600 6067 50  0000 C CNN
 F 1 "RST_FE2.1" H 3600 5976 50  0000 C CNN
 F 2 "LCSC:Switch_4_4_1.7_C10852" H 3600 5800 50  0001 C CNN
@@
 P 3300 6050
 AR Path="/5B3365B6/5BBA4BC7" Ref="#PWR?"  Part="1"
-AR Path="/5B3365B0/5BBA4BC7" Ref="#PWR?"  Part="1"
-F 0 "#PWR?" H 3300 5800 50  0001 C CNN
+AR Path="/5B3365B0/5BBA4BC7" Ref="#PWR0106"  Part="1"
+F 0 "#PWR0106" H 3300 5800 50  0001 C CNN
 F 1 "GND" H 3305 5877 50  0000 C CNN
 F 2 "" H 3300 6050 50  0001 C CNN
@@
 	3300 5800 3300 6050
 $Comp
-L Mister_Logo:Logo L?
+L Mister_Logo:Logo L1
 U 1 1 5BBB1048
 P 9800 2050
-F 0 "L?" H 9978 2096 50  0000 L CNN
+F 0 "L1" H 9978 2096 50  0000 L CNN
 F 1 "Logo" H 9978 2005 50  0000 L CNN
 F 2 "DE10:MiSTer_Logo" H 9800 2050 50  0001 C CNN
@@
 	1    0    0    -1
 $EndComp
+Text Label 3900 5800 0    50   ~ 0
+FE_2_1_RST
+Text Label 5850 4800 0    50   ~ 0
+VDD3_3_FE21
 $EndSCHEMATC
